File: hardware/hardware.kicad_pcb (KiCad board)
At the start: 2 copper layers, 25.7 x 34.4 mm, 3 parts, among them P1 CONN_01X08, P2 CONN_01X08

Commit message: 1s SweetTime v2 version
Parts:
- added C1: 10n, Capacitors_SMD:C_0402, F.Cu at (131.1, 105.4)
- added D1: WS2812B, WS2812B:LED_WS2812B, F.Cu at (135.1, 91.9)
- added D2: WS2812B, WS2812B:LED_WS2812B, F.Cu at (142.2, 88.6)
- added D3: WS2812B, WS2812B:LED_WS2812B, F.Cu at (142.2, 95.2)
- added D4: 1N4004, Diodes_ThroughHole:Diode_DO-35_SOD27_Horizontal_RM10, F.Cu at (140.7, 99.3)
- added P3: CONN_01X02, Connect:PINHEAD1-2, F.Cu at (132.3, 109.5)
- added R1: 10K, Resistors_SMD:R_0402, F.Cu at (133.6, 105.4)
Connections:
- P1 pad 2: /GND -> GND
Routing:
- net /+5V: track 0.00 -> 35.0 mm
- net /D6: track 0.00 -> 27.8 mm, vias 0 -> 1
- net /D5: track 0.00 -> 23.6 mm
- net Net-(D2-Pad2): track 0.00 -> 8.40 mm
- net Net-(D1-Pad1): track 0.00 -> 7.81 mm
- net /D2: track 0.00 -> 5.29 mm
- net GND: track 0.00 -> 4.75 mm
- net Net-(D1-Pad2): track 0.00 -> 2.25 mm
- added copper zone on F.Cu, net GND
Other:
- board text added: "SweetTime"
- board text added: "u.dinask.eu/trender"
