File: hardware/hardware.kicad_pcb (KiCad board)
At the start: 2 copper layers, 25.7 x 34.4 mm, 13 parts, among them P1 CONN_01X08, P2 CONN_01X08, P3 CONN_01X02, P4 CONN_01X03

Commit message: change pinheader face for better 3D display
Parts:
- P1, P2: moved to B.Cu
- turned P1 to 0 degrees
- turned P2 to 0 degrees
Changed lines of the file:
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@@
     (add_net "Net-(D3-Pad2)")
   )
-  (module D1_mini:D1_mini_Pin_Header (layer F.Cu)
-    (at 127.49 103.95 180)
+  (module D1_mini:D1_mini_Pin_Header (layer B.Cu)
+    (at 127.49 103.95)
     (descr "Through hole pin header")
     (tags "pin header")
-    (fp_text reference P1 (at -0.11 -2.45 180) (layer F.SilkS) hide
-      (effects (font (size 1 1) (thickness 0.15)))
-    )
-    (fp_text value CONN_01X08 (at 0 -3.1 180) (layer F.Fab) hide
-      (effects (font (size 1 1) (thickness 0.15)))
-    )
-    (fp_line (start -1.75 -1.75) (end -1.75 19.55) (layer F.CrtYd) (width 0.05))
-    (fp_line (start 1.75 -1.75) (end 1.75 19.55) (layer F.CrtYd) (width 0.05))
-    (fp_line (start -1.75 -1.75) (end 1.75 -1.75) (layer F.CrtYd) (width 0.05))
-    (fp_line (start -1.75 19.55) (end 1.75 19.55) (layer F.CrtYd) (width 0.05))
-    (pad 1 thru_hole rect (at 0 0 180) (size 1.8 1.8) (drill 1.016) (layers *.Cu *.Mask F.SilkS)
+    (fp_text reference P1 (at -0.11 2.45) (layer B.SilkS) hide
+      (effects (font (size 1 1) (thickness 0.15)) (justify mirror))
+    )
+    (fp_text value CONN_01X08 (at 0 3.1) (layer B.Fab) hide
+      (effects (font (size 1 1) (thickness 0.15)) (justify mirror))
+    )
+    (fp_line (start -1.75 1.75) (end -1.75 -19.55) (layer B.CrtYd) (width 0.05))
+    (fp_line (start 1.75 1.75) (end 1.75 -19.55) (layer B.CrtYd) (width 0.05))
+    (fp_line (start -1.75 1.75) (end 1.75 1.75) (layer B.CrtYd) (width 0.05))
+    (fp_line (start -1.75 -19.55) (end 1.75 -19.55) (layer B.CrtYd) (width 0.05))
+    (pad 1 thru_hole rect (at 0 0) (size 1.8 1.8) (drill 1.016) (layers *.Cu *.Mask B.SilkS)
       (net 1 /+5V))
-    (pad 2 thru_hole oval (at 0 2.54 180) (size 1.8 1.8) (drill 1.016) (layers *.Cu *.Mask F.SilkS)
+    (pad 2 thru_hole oval (at 0 -2.54) (size 1.8 1.8) (drill 1.016) (layers *.Cu *.Mask B.SilkS)
       (net 16 GND))
-    (pad 3 thru_hole oval (at 0 5.08 180) (size 1.8 1.8) (drill 1.016) (layers *.Cu *.Mask F.SilkS)
+    (pad 3 thru_hole oval (at 0 -5.08) (size 1.8 1.8) (drill 1.016) (layers *.Cu *.Mask B.SilkS)
       (net 2 /D4))
-    (pad 4 thru_hole oval (at 0 7.62 180) (size 1.8 1.8) (drill 1.016) (layers *.Cu *.Mask F.SilkS)
+    (pad 4 thru_hole oval (at 0 -7.62) (size 1.8 1.8) (drill 1.016) (layers *.Cu *.Mask B.SilkS)
       (net 3 /D3))
-    (pad 5 thru_hole oval (at 0 10.16 180) (size 1.8 1.8) (drill 1.016) (layers *.Cu *.Mask F.SilkS)
+    (pad 5 thru_hole oval (at 0 -10.16) (size 1.8 1.8) (drill 1.016) (layers *.Cu *.Mask B.SilkS)
       (net 4 /D2))
-    (pad 6 thru_hole oval (at 0 12.7 180) (size 1.8 1.8) (drill 1.016) (layers *.Cu *.Mask F.SilkS)
+    (pad 6 thru_hole oval (at 0 -12.7) (size 1.8 1.8) (drill 1.016) (layers *.Cu *.Mask B.SilkS)
       (net 5 /D1))
-    (pad 7 thru_hole oval (at 0 15.24 180) (size 1.8 1.8) (drill 1.016) (layers *.Cu *.Mask F.SilkS)
+    (pad 7 thru_hole oval (at 0 -15.24) (size 1.8 1.8) (drill 1.016) (layers *.Cu *.Mask B.SilkS)
       (net 6 /RX))
-    (pad 8 thru_hole oval (at 0 17.78 180) (size 1.8 1.8) (drill 1.016) (layers *.Cu *.Mask F.SilkS)
+    (pad 8 thru_hole oval (at 0 -17.78) (size 1.8 1.8) (drill 1.016) (layers *.Cu *.Mask B.SilkS)
       (net 7 /TX))
     (model Pin_Headers.3dshapes/Pin_Header_Straight_1x08.wrl
@@
     )
   )
-  (module D1_mini:D1_mini_Pin_Header (layer F.Cu)
-    (at 150.35 103.95 180)
+  (module D1_mini:D1_mini_Pin_Header (layer B.Cu)
+    (at 150.35 103.95)
     (descr "Through hole pin header")
     (tags "pin header")
-    (fp_text reference P2 (at 0.05 20.15 180) (layer F.SilkS) hide
-      (effects (font (size 1 1) (thickness 0.15)))
-    )
-    (fp_text value CONN_01X08 (at 0 -3.1 180) (layer F.Fab) hide
-      (effects (font (size 1 1) (thickness 0.15)))
-    )
-    (fp_line (start -1.75 -1.75) (end -1.75 19.55) (layer F.CrtYd) (width 0.05))
-    (fp_line (start 1.75 -1.75) (end 1.75 19.55) (layer F.CrtYd) (width 0.05))
-    (fp_line (start -1.75 -1.75) (end 1.75 -1.75) (layer F.CrtYd) (width 0.05))
-    (fp_line (start -1.75 19.55) (end 1.75 19.55) (layer F.CrtYd) (width 0.05))
-    (pad 1 thru_hole rect (at 0 0 180) (size 1.8 1.8) (drill 1.016) (layers *.Cu *.Mask F.SilkS)
+    (fp_text reference P2 (at 0.05 -20.15) (layer B.SilkS) hide
+      (effects (font (size 1 1) (thickness 0.15)) (justify mirror))
+    )
+    (fp_text value CONN_01X08 (at 0 3.1) (layer B.Fab) hide
+      (effects (font (size 1 1) (thickness 0.15)) (justify mirror))
+    )
+    (fp_line (start -1.75 1.75) (end -1.75 -19.55) (layer B.CrtYd) (width 0.05))
+    (fp_line (start 1.75 1.75) (end 1.75 -19.55) (layer B.CrtYd) (width 0.05))
+    (fp_line (start -1.75 1.75) (end 1.75 1.75) (layer B.CrtYd) (width 0.05))
+    (fp_line (start -1.75 -19.55) (end 1.75 -19.55) (layer B.CrtYd) (width 0.05))
+    (pad 1 thru_hole rect (at 0 0) (size 1.8 1.8) (drill 1.016) (layers *.Cu *.Mask B.SilkS)
       (net 8 /+3.3V))
-    (pad 2 thru_hole oval (at 0 2.54 180) (size 1.8 1.8) (drill 1.016) (layers *.Cu *.Mask F.SilkS)
+    (pad 2 thru_hole oval (at 0 -2.54) (size 1.8 1.8) (drill 1.016) (layers *.Cu *.Mask B.SilkS)
       (net 9 /D8))
-    (pad 3 thru_hole oval (at 0 5.08 180) (size 1.8 1.8) (drill 1.016) (layers *.Cu *.Mask F.SilkS)
+    (pad 3 thru_hole oval (at 0 -5.08) (size 1.8 1.8) (drill 1.016) (layers *.Cu *.Mask B.SilkS)
       (net 10 /D7))
-    (pad 4 thru_hole oval (at 0 7.62 180) (size 1.8 1.8) (drill 1.016) (layers *.Cu *.Mask F.SilkS)
+    (pad 4 thru_hole oval (at 0 -7.62) (size 1.8 1.8) (drill 1.016) (layers *.Cu *.Mask B.SilkS)
       (net 11 /D6))
-    (pad 5 thru_hole oval (at 0 10.16 180) (size 1.8 1.8) (drill 1.016) (layers *.Cu *.Mask F.SilkS)
+    (pad 5 thru_hole oval (at 0 -10.16) (size 1.8 1.8) (drill 1.016) (layers *.Cu *.Mask B.SilkS)
       (net 12 /D5))
-    (pad 6 thru_hole oval (at 0 12.7 180) (size 1.8 1.8) (drill 1.016) (layers *.Cu *.Mask F.SilkS)
+    (pad 6 thru_hole oval (at 0 -12.7) (size 1.8 1.8) (drill 1.016) (layers *.Cu *.Mask B.SilkS)
       (net 13 /D0))
-    (pad 7 thru_hole oval (at 0 15.24 180) (size 1.8 1.8) (drill 1.016) (layers *.Cu *.Mask F.SilkS)
+    (pad 7 thru_hole oval (at 0 -15.24) (size 1.8 1.8) (drill 1.016) (layers *.Cu *.Mask B.SilkS)
       (net 14 /A0))
-    (pad 8 thru_hole oval (at 0 17.78 180) (size 1.8 1.8) (drill 1.016) (layers *.Cu *.Mask F.SilkS)
+    (pad 8 thru_hole oval (at 0 -17.78) (size 1.8 1.8) (drill 1.016) (layers *.Cu *.Mask B.SilkS)
       (net 15 /RST))
     (model Pin_Headers.3dshapes/Pin_Header_Straight_1x08.wrl
@@
   (segment (start 141.668 103.95) (end 150.35 103.95) (width 0.25) (layer F.Cu) (net 8))
   (segment (start 140.208 105.41) (end 141.668 103.95) (width 0.25) (layer F.Cu) (net 8))
+  (segment (start 134.366 103.378) (end 133.154 104.59) (width 0.25) (layer F.Cu) (net 12))
+  (segment (start 133.154 104.59) (end 133.154 105.41) (width 0.25) (layer F.Cu) (net 12))
   (segment (start 150.35 93.79) (end 149.796 93.79) (width 0.25) (layer F.Cu) (net 12))
   (segment (start 149.796 93.79) (end 148.082 95.504) (width 0.25) (layer F.Cu) (net 12))
@@
   (segment (start 148.082 101.346) (end 146.05 103.378) (width 0.25) (layer F.Cu) (net 12))
   (segment (start 146.05 103.378) (end 134.366 103.378) (width 0.25) (layer F.Cu) (net 12))
-  (segment (start 134.366 103.378) (end 133.154 104.59) (width 0.25) (layer F.Cu) (net 12))
-  (segment (start 133.154 104.59) (end 133.154 105.41) (width 0.25) (layer F.Cu) (net 12))
   (segment (start 133.154 105.41) (end 133.154 109.024) (width 0.25) (layer F.Cu) (net 12))
   (segment (start 133.154 109.024) (end 133.604 109.474) (width 0.25) (layer F.Cu) (net 12))
