File: hardware/hardware.sch (KiCad schematic (older format))
At the start: 2 parts, among them P1 CONN_01X08, P2 CONN_01X08

Commit message: 1s SweetTime v2 version
Parts:
- added C1: 10n, Capacitors_SMD:C_0402, symbol C
- added D1, D2, D3: WS2812B, WS2812B:LED_WS2812B, symbol WS2812B
- added D4: 1N4004, Diodes_ThroughHole:Diode_DO-35_SOD27_Horizontal_RM10, symbol D
- added P3: CONN_01X02, Connect:PINHEAD1-2, symbol CONN_01X02
- added R1: 10K, Resistors_SMD:R_0402, symbol R
Connections:
- net +5V: now also D2.1 (VDD), D3.1 (VDD), D4.2 (A)
- net D2: now also D1.4 (DIN)
- net D5: now also R1.1
- net D6: now also C1.1, P3.1 (P1), R1.2
- net GND: now also C1.2, D1.3 (VSS), D2.3 (VSS), D3.3 (VSS), P3.2 (P2)
- new net: D1.1 (VDD), D4.1 (K)
- new net: D1.2 (DOUT), D2.4 (DIN)
- new net: D2.2 (DOUT), D3.4 (DIN)
- no-connect marks 0 -> 11
Other:
- note added: "Control button connector"
- note added: "RGB leds"
Changed lines of the file:
@@
 LIBS:contrib
 LIBS:valves
+LIBS:WS2812B
 LIBS:hardware-cache
 EELAYER 25 0
@@
 Text Notes 8550 600  0    60   ~ 0
 D1 Mini Shield
+$Comp
+L WS2812B D1
+U 1 1 577173C5
+P 1500 1800
+F 0 "D1" H 1100 2250 50  0000 L CNN
+F 1 "WS2812B" H 1100 1300 50  0000 L CNN
+F 2 "WS2812B:LED_WS2812B" H 1500 1800 50  0001 L CNN
+F 3 "" H 1500 1800 60  0000 C CNN
+	1    1500 1800
+	1    0    0    -1
+$EndComp
+$Comp
+L WS2812B D2
+U 1 1 577174D3
+P 3050 1800
+F 0 "D2" H 2650 2250 50  0000 L CNN
+F 1 "WS2812B" H 2650 1300 50  0000 L CNN
+F 2 "WS2812B:LED_WS2812B" H 3050 1800 50  0001 L CNN
+F 3 "" H 3050 1800 60  0000 C CNN
+	1    3050 1800
+	1    0    0    -1
+$EndComp
+$Comp
+L WS2812B D3
+U 1 1 57717547
+P 4600 1800
+F 0 "D3" H 4200 2250 50  0000 L CNN
+F 1 "WS2812B" H 4200 1300 50  0000 L CNN
+F 2 "WS2812B:LED_WS2812B" H 4600 1800 50  0001 L CNN
+F 3 "" H 4600 1800 60  0000 C CNN
+	1    4600 1800
+	1    0    0    -1
+$EndComp
+Wire Wire Line
+	3650 1800 4000 1800
+Wire Wire Line
+	2100 1800 2450 1800
+$Comp
+L D D4
+U 1 1 57717974
+P 2100 950
+F 0 "D4" H 2100 1050 50  0000 C CNN
+F 1 "1N4004" H 2100 850 50  0000 C CNN
+F 2 "Diodes_ThroughHole:Diode_DO-35_SOD27_Horizontal_RM10" H 2100 950 60  0001 C CNN
+F 3 "" H 2100 950 60  0000 C CNN
+	1    2100 950
+	0    -1   -1   0
+$EndComp
+Wire Wire Line
+	2100 1500 2100 1100
+Wire Wire Line
+	2100 800  5200 800
+Wire Wire Line
+	3650 800  3650 1500
+Wire Wire Line
+	5200 800  5200 1500
+Connection ~ 3650 800
+Text Label 2100 800  2    60   ~ 0
++5V
+NoConn ~ 5200 1800
+Wire Wire Line
+	2100 2100 2100 2550
+Wire Wire Line
+	2100 2550 5200 2550
+Wire Wire Line
+	3650 2550 3650 2100
+Wire Wire Line
+	5200 2550 5200 2100
+Connection ~ 3650 2550
+Text Label 2100 2550 2    60   ~ 0
+GND
+$Comp
+L R R1
+U 1 1 57717D17
+P 6550 1000
+F 0 "R1" V 6630 1000 50  0000 C CNN
+F 1 "10K" V 6550 1000 50  0000 C CNN
+F 2 "Resistors_SMD:R_0402" V 6480 1000 30  0001 C CNN
+F 3 "" H 6550 1000 30  0000 C CNN
+	1    6550 1000
+	1    0    0    -1
+$EndComp
+$Comp
+L C C1
+U 1 1 57717D66
+P 6550 1550
+F 0 "C1" H 6575 1650 50  0000 L CNN
+F 1 "10n" H 6575 1450 50  0000 L CNN
+F 2 "Capacitors_SMD:C_0402" H 6588 1400 30  0001 C CNN
+F 3 "" H 6550 1550 60  0000 C CNN
+	1    6550 1550
+	1    0    0    -1
+$EndComp
+$Comp
+L GND #PWR01
+U 1 1 57717E9A
+P 10500 6100
+F 0 "#PWR01" H 10500 5850 50  0001 C CNN
+F 1 "GND" H 10500 5950 50  0000 C CNN
+F 2 "" H 10500 6100 60  0000 C CNN
+F 3 "" H 10500 6100 60  0000 C CNN
+	1    10500 6100
+	1    0    0    -1
+$EndComp
+$Comp
+L PWR_FLAG #FLG02
+U 1 1 57717ED2
+P 10500 6000
+F 0 "#FLG02" H 10500 6095 50  0001 C CNN
+F 1 "PWR_FLAG" H 10500 6180 50  0000 C CNN
+F 2 "" H 10500 6000 60  0000 C CNN
+F 3 "" H 10500 6000 60  0000 C CNN
+	1    10500 6000
+	1    0    0    -1
+$EndComp
+Text Label 10500 6050 2    60   ~ 0
+GND
+Wire Wire Line
+	10500 6000 10500 6100
+$Comp
+L PWR_FLAG #FLG03
+U 1 1 57718046
+P 10900 6000
+F 0 "#FLG03" H 10900 6095 50  0001 C CNN
+F 1 "PWR_FLAG" H 10900 6180 50  0000 C CNN
+F 2 "" H 10900 6000 60  0000 C CNN
+F 3 "" H 10900 6000 60  0000 C CNN
+	1    10900 6000
+	1    0    0    -1
+$EndComp
+$Comp
+L PWR_FLAG #FLG04
+U 1 1 5771806C
+P 10100 6000
+F 0 "#FLG04" H 10100 6095 50  0001 C CNN
+F 1 "PWR_FLAG" H 10100 6180 50  0000 C CNN
+F 2 "" H 10100 6000 60  0000 C CNN
+F 3 "" H 10100 6000 60  0000 C CNN
+	1    10100 6000
+	1    0    0    -1
+$EndComp
+Wire Wire Line
+	10100 6000 10100 6100
+Wire Wire Line
+	10900 6000 10900 6100
+Text Label 10100 6100 2    60   ~ 0
++5V
+Text Label 10900 6100 2    60   ~ 0
++3.3V
+Wire Notes Line
+	9700 6500 9700 5500
+Wire Notes Line
+	9700 5500 11200 5500
+Wire Notes Line
+	500  3350 5800 3350
+Wire Notes Line
+	5800 3350 5800 500
+Wire Wire Line
+	6550 1150 6550 1400
+Wire Wire Line
+	6200 1300 6950 1300
+Connection ~ 6550 1300
+Wire Wire Line
+	6550 1700 6550 2100
+Wire Wire Line
+	6550 1900 6200 1900
+Connection ~ 6550 1900
+$Comp
+L GND #PWR05
+U 1 1 5771843C
+P 6550 2100
+F 0 "#PWR05" H 6550 1850 50  0001 C CNN
+F 1 "GND" H 6550 1950 50  0000 C CNN
+F 2 "" H 6550 2100 60  0000 C CNN
+F 3 "" H 6550 2100 60  0000 C CNN
+	1    6550 2100
+	1    0    0    -1
+$EndComp
+$Comp
+L GND #PWR06
+U 1 1 5771848D
+P 3650 2550
+F 0 "#PWR06" H 3650 2300 50  0001 C CNN
+F 1 "GND" H 3650 2400 50  0000 C CNN
+F 2 "" H 3650 2550 60  0000 C CNN
+F 3 "" H 3650 2550 60  0000 C CNN
+	1    3650 2550
+	1    0    0    -1
+$EndComp
+Wire Notes Line
+	5850 2650 7400 2650
+Wire Notes Line
+	7400 2650 7400 450
+Text Notes 550  3250 0    60   ~ 0
+RGB leds
+Text Notes 5850 2600 0    60   ~ 0
+Control button connector
+$Comp
+L CONN_01X02 P3
+U 1 1 577189A7
+P 6000 1600
+F 0 "P3" H 6000 1750 50  0000 C CNN
+F 1 "CONN_01X02" V 6100 1600 50  0000 C CNN
+F 2 "Connect:PINHEAD1-2" H 6000 1600 60  0001 C CNN
+F 3 "" H 6000 1600 60  0000 C CNN
+	1    6000 1600
+	-1   0    0    -1
+$EndComp
+Wire Wire Line
+	6200 1300 6200 1550
+Wire Wire Line
+	6200 1900 6200 1650
+Text Label 900  1800 2    60   ~ 0
+D2
+Text Label 6550 850  0    60   ~ 0
+D5
+Text Label 6950 1300 0    60   ~ 0
+D6
+NoConn ~ 9450 1250
+NoConn ~ 9450 1350
+NoConn ~ 9450 1550
+NoConn ~ 9450 1650
+NoConn ~ 9450 1750
+NoConn ~ 10300 1150
+NoConn ~ 10300 1250
+NoConn ~ 10300 1550
+NoConn ~ 10300 1650
+NoConn ~ 10300 1750
 $EndSCHEMATC
